File: CAD/output_controller/output_controller.sch (KiCad schematic (older format))
At the start: 71 parts

Commit message: progress on charge and output layout
Parts:
- added MK1, MK2, MK3, MK4: Mounting_Hole, MountingHole:MountingHole_4.3mm_M4, symbol Mechanical:Mounting_Hole
- C1: renamed from C?; footprint (none) -> Capacitor_SMD:C_1206_3216Metric
- C2, C3, C4, C5: renamed from C?; footprint (none) -> Capacitor_SMD:C_0603_1608Metric
- D1, D2, D3: renamed from D?; footprint (none) -> Diode_SMD:D_SOD-523
- F1: renamed from F?; footprint (none) -> Fuse:Fuseholder_Blade_Mini_Keystone_3568
- J2: renamed from J?; footprint Connector_Phoenix_MC:PhoenixContact_MCV_1,5_2-G-5.08_1x02_P5.08mm_Vertical -> Connector_PinHeader_2.54mm:PinHeader_1x02_P2.54mm_Vertical
- J3, J4: renamed from J?; footprint (none) -> Connector_PinHeader_2.54mm:PinHeader_1x05_P2.54mm_Vertical
- Q1, Q3: renamed from Q?; footprint (none) -> Package_TO_SOT_SMD:TO-252-2
- Q4, Q5, Q6, Q7: renamed from Q?; footprint (none) -> Package_TO_SOT_SMD:SOT-23
- R1, R14, R2, R3, R4, R5: renamed from R?; footprint (none) -> Resistor_SMD:R_0603_1608Metric
- R10, R11, R12, R13, R15, R16, R17, R18, R19, R20, R21, R22, R23, R24, R25, R26, R27, R28, R29, R30, R31, R32, R33, R34, R6, R7, R8, R9: renamed from R?; footprint Resistor_SMD:R_0402_1005Metric -> Resistor_SMD:R_0603_1608Metric
- SW1: renamed from SW?; footprint (none) -> Connector_PinHeader_2.54mm:PinHeader_1x02_P2.54mm_Vertical
- SW2, SW3, SW4, SW5: renamed from SW?; footprint (none) -> Connector_PinHeader_2.54mm:PinHeader_1x04_P2.54mm_Vertical
- gave numbers to parts that had none: 14
Connections:
- wire segments 245 -> 246

Commit message: finishes output board
Connections:
- net labels added: IN1, IN2, IN3, IN4, IN_SW1, IN_SW2, IN_SW3, IN_SW4, IS1, IS2, IS3, IS4, OUT1, OUT2, OUT3, OUT4, VBB, VIN, VIN_FUSED, VIN_VBB
Changed lines of the file:
@@
 	1    0    0    -1
 $EndComp
-Wire Wire Line
-	7450 2850 7750 2850
 $Comp
 L Device:D_Zener_Small D4
@@
 F 3 "~" H 2300 3550 50  0001 C CNN
 	1    2300 3550
-	-1   0    0    -1
+	-1   0    0    1
 $EndComp
 $Comp
@@
 	6450 3050 6450 3200
 Wire Wire Line
-	7550 2550 9750 2550
+	7550 2550 7750 2550
 $Comp
 L Device:R_Small R19
@@
 Wire Wire Line
 	7750 3150 7750 3250
-Wire Wire Line
-	7750 2950 7750 2850
-Connection ~ 7750 2850
-Wire Wire Line
-	7750 2850 8300 2850
 $Comp
 L Mechanical:Mounting_Hole MK1
@@
 Wire Wire Line
 	3700 2000 3700 2050
+Text Label 2600 1350 0    50   ~ 0
+VIN
+Text Label 3200 1350 0    50   ~ 0
+VIN_FUSED
+Text Label 5400 1350 0    50   ~ 0
+VBB
+Text Label 8050 2550 0    50   ~ 0
+OUT1
+Text Label 7950 2850 0    50   ~ 0
+IS1
+Text Label 6450 2650 0    50   ~ 0
+IN1
+Text Label 6100 3050 0    50   ~ 0
+IN_SW1
+Text Label 7850 4500 0    50   ~ 0
+OUT2
+Text Label 7850 4800 0    50   ~ 0
+IS2
+Text Label 6450 4600 0    50   ~ 0
+IN2
+Text Label 6100 5000 0    50   ~ 0
+IN_SW2
+Text Label 7950 6500 0    50   ~ 0
+OUT3
+Text Label 7950 6800 0    50   ~ 0
+IS3
+Text Label 6450 6600 0    50   ~ 0
+IN3
+Text Label 6100 7000 0    50   ~ 0
+IN_SW3
+Text Label 7950 8550 0    50   ~ 0
+OUT4
+Text Label 7950 8850 0    50   ~ 0
+IS4
+Text Label 6450 8650 0    50   ~ 0
+IN4
+Text Label 6100 9050 0    50   ~ 0
+IN_SW4
+Text Label 4500 1350 0    50   ~ 0
+VIN_VBB
+Wire Wire Line
+	7450 2850 8300 2850
+Wire Wire Line
+	7750 2950 7750 2550
+Connection ~ 7750 2550
+Wire Wire Line
+	7750 2550 9750 2550
 $EndSCHEMATC
