File: CAD/output_controller/output_controller.kicad_pcb (KiCad board)
At the start: 2 copper layers, 50 x 100 mm, 75 parts, among them J1 12V_IN, J2 MCU_SW, J3 MCU_EN, J4 MCU_IS, J5 12V_A, J6 12V_A, J7 12V_A, J8 12V_A, Q1 Q_PMOS_GDS, Q2 MMBT3904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

Commit message: finishes output board
Parts:
- moved R19 39.8 mm to (107.0, 90.0), turned to 0 degrees
- moved C3 34.1 mm to (107.0, 94.5), turned to 0 degrees
- moved C5 33.1 mm to (107.0, 122.0), turned to 0 degrees
- moved R15 32.0 mm to (111.2, 85.0), turned to 180 degrees
- moved R16 30.1 mm to (111.0, 98.0), turned to 180 degrees
- moved R18 29.3 mm to (111.0, 125.0), turned to 180 degrees
- moved C4 14.1 mm to (107.0, 107.5), turned to 0 degrees
- moved R17 14.1 mm to (111.0, 110.5)
- moved R10 11.7 mm to (122.5, 140.2)
- moved R6 11.7 mm to (122.5, 144.2)
- moved R23 9.22 mm to (142.0, 80.0)
- moved R27 9.22 mm to (138.0, 77.0)
- moved R28 9.22 mm to (142.0, 77.0)
- moved R24 8.25 mm to (141.0, 101.0)
- moved R29 8.25 mm to (136.8, 98.0)
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Connections:
- net Net-(C1-Pad1) renamed /VIN_FUSED
- net Net-(C2-Pad1) renamed /IN_SW1
- net Net-(C3-Pad1) renamed /IN_SW2
- net Net-(C4-Pad1) renamed /IN_SW3
- net Net-(C5-Pad1) renamed /IN_SW4
- net Net-(D2-Pad1) renamed /VIN_VBB
- net Net-(D3-Pad2) renamed /VBB
- net Net-(F1-Pad2) renamed /VIN
- net Net-(J6-Pad1) renamed /OUT2
- net Net-(J7-Pad1) renamed /OUT3
- net Net-(J8-Pad1) renamed /OUT4
- net Net-(R15-Pad1) renamed /IN1
- net Net-(R16-Pad1) renamed /IN2
- net Net-(R17-Pad1) renamed /IN3
- net Net-(R18-Pad1) renamed /IN4
- net Net-(R24-Pad1) renamed /IS2
- net Net-(R25-Pad1) renamed /IS3
- net Net-(R26-Pad1) renamed /IS4
- J3 pad 1: /ch1_en -> GND
- J3 pad 2: /ch2_en -> /ch4_en
- J3 pad 4: /ch4_en -> /ch2_en
- J3 pad 5: GND -> /ch1_en
- J5 pad 1: Net-(J5-Pad1) -> /OUT1
- R19 pad 2: Net-(R19-Pad2) -> /OUT1
- R23 pad 1: Net-(R19-Pad2) -> /IS1
- R27 pad 2: Net-(R19-Pad2) -> /IS1
- R28 pad 2: Net-(R19-Pad2) -> /IS1
- U1 pad 1: Net-(J5-Pad1) -> /OUT1
- U1 pad 4: Net-(R19-Pad2) -> /IS1
- U1 pad 5: Net-(J5-Pad1) -> /OUT1
Routing:
- net /ch1_i: track 0.00 -> 82.0 mm, vias 0 -> 2
- net Net-(Q4-Pad1): track 0.00 -> 65.3 mm
- net /ch2_i: track 0.00 -> 62.6 mm, vias 0 -> 2
- net Net-(Q5-Pad1): track 0.00 -> 54.0 mm
- net Net-(D1-Pad1): track 0.00 -> 53.6 mm
- net GND: track 0.00 -> 47.7 mm, vias 0 -> 17
- net /ch3_i: track 0.00 -> 43.7 mm, vias 0 -> 2
- net /IN1: track 0.00 -> 40.0 mm, vias 0 -> 2
- net /OUT1: track 0.00 -> 39.6 mm, vias 0 -> 4
- net Net-(Q6-Pad1): track 0.00 -> 35.7 mm
- net /OUT2: track 0.00 -> 35.7 mm, vias 0 -> 4
- net /OUT4: track 0.00 -> 33.9 mm, vias 0 -> 4
- net /IN4: track 0.00 -> 33.7 mm, vias 0 -> 4
- net /IN2: track 0.00 -> 33.2 mm, vias 0 -> 4
- net /OUT3: track 0.00 -> 33.0 mm, vias 0 -> 4
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- added copper zone on F.Cu, net /OUT1
- added copper zone on F.Cu, net /OUT2
- added copper zone on F.Cu, net /OUT3
- added copper zone on F.Cu, net /OUT4
- added copper zone on F.Cu, net /VBB
- added copper zone on F.Cu, net /VIN
- added copper zone on F.Cu, net /VIN_FUSED
- added copper zone on F.Cu, net /VIN_VBB
- added copper zone on B.Cu, net GND
Other:
- net class PWR added: clearance 0.2, trace_width 0.5, via_dia 0.8, via_drill 0.4

Commit message: finishes layout for mcu controller
Routing:
- net Net-(Q7-Pad1): track 21.8 -> 22.9 mm

Commit message: finishes output controller
Other:
- board text added: "CH1_EN"
- board text added: "CH1_I"
- board text added: "CH2_EN"
- board text added: "CH2_I"
- board text added: "CH3_EN"
- board text added: "CH3_I"
- board text added: "CH4_EN"
- board text added: "CH4_I"
- board text added: "GND"
- board text added: "LED1"
- board text added: "LED2"
- board text added: "LED3"
- board text added: "LED4"
- board text added: "MCU_EN"
- board text added: "ON_SW"
- board text added: "OUT1"
- board text added: "OUT2"
- board text added: "OUT3"
- board text added: "OUT4"
- board text added: "OUTPUT CONTROLLER 1.0V 180530 FITZ"
- board text added: "SW1"
- board text added: "SW2"
- board text added: "SW3"
- board text added: "SW4"
- board text added: "VIN"
