File: CAD/mcu_controller/mcu_controller.kicad_pcb (KiCad board)
At the start: 2 copper layers, 100 x 50 mm, 81 parts, among them J1 BATT, J10 out2_ch_en, J11 SPI, J12 I2C, J13 chrg1_ctrl, J14 chrg2_ctrl, J15 chrg3_ctrl, J16 out1_en, J17 out2_en, J19 UART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

Commit message: removes pin 17 connection to VIN on mcu controller
Connections:
- U3 pad 15: +5V -> Net-(U3-Pad15)
Changed lines of the file:
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@@
     (zones 0)
     (modules 81)
-    (nets 93)
+    (nets 94)
   )
   (page A4)
@@
   (net 91 /I2C_SDA)
   (net 92 /I2C_SCL)
+  (net 93 "Net-(U3-Pad15)")
   (net_class Default "This is the default net class."
     (clearance 0.25)
@@
     (add_net "Net-(R7-Pad1)")
     (add_net "Net-(R9-Pad1)")
+    (add_net "Net-(U3-Pad15)")
     (add_net "Net-(U3-Pad16)")
     (add_net "Net-(U3-Pad34)")
@@
       (net 6 /MISO))
     (pad 15 thru_hole circle (at 16.51 5.08) (size 1.6 1.6) (drill 1.1) (layers *.Cu *.Mask F.SilkS)
-      (net 5 +5V))
+      (net 93 "Net-(U3-Pad15)"))
     (pad 16 thru_hole circle (at 16.51 2.54) (size 1.6 1.6) (drill 1.1) (layers *.Cu *.Mask F.SilkS)
       (net 4 "Net-(U3-Pad16)"))
@@
   (segment (start 112.07 111) (end 111 111) (width 0.5) (layer F.Cu) (net 1))
   (segment (start 111 111) (end 110.5 111.5) (width 0.5) (layer F.Cu) (net 1))
+  (segment (start 187.96 126.96) (end 188 127) (width 0.25) (layer F.Cu) (net 1))
+  (segment (start 193.04 121.92) (end 198 121.92) (width 0.5) (layer B.Cu) (net 1))
+  (segment (start 187.96 127) (end 193.04 121.92) (width 0.5) (layer B.Cu) (net 1))
   (segment (start 181.9 147.02) (end 182.88 148) (width 0.25) (layer F.Cu) (net 2))
   (segment (start 181.9 144.5) (end 181.9 147.02) (width 0.25) (layer F.Cu) (net 2))
@@
   (segment (start 185.42 137.16) (end 186.734999 135.845001) (width 0.25) (layer F.Cu) (net 3))
   (segment (start 194.234999 138.385001) (end 192.2 138.385001) (width 0.25) (layer F.Cu) (net 3))
+  (segment (start 184.570001 136.310001) (end 185.42 137.16) (width 0.25) (layer F.Cu) (net 3))
+  (segment (start 170.577994 121.724998) (end 182.372002 121.724998) (width 0.25) (layer F.Cu) (net 3))
+  (segment (start 183.194978 132.540852) (end 184.175013 133.520887) (width 0.25) (layer F.Cu) (net 3))
+  (segment (start 166.51 117.38) (end 167.309999 118.179999) (width 0.25) (layer F.Cu) (net 3))
+  (segment (start 184.175013 133.520887) (end 184.175013 135.915013) (width 0.25) (layer F.Cu) (net 3))
+  (segment (start 184.175013 135.915013) (end 184.570001 136.310001) (width 0.25) (layer F.Cu) (net 3))
+  (segment (start 182.372002 121.724998) (end 183.194978 122.547974) (width 0.25) (layer F.Cu) (net 3))
+  (segment (start 183.194978 122.547974) (end 183.194978 132.540852) (width 0.25) (layer F.Cu) (net 3))
+  (segment (start 167.309999 118.457003) (end 170.577994 121.724998) (width 0.25) (layer F.Cu) (net 3))
+  (segment (start 167.309999 118.179999) (end 167.309999 118.457003) (width 0.25) (layer F.Cu) (net 3))
   (segment (start 120.07 116.5) (end 120.5 116.07) (width 0.5) (layer F.Cu) (net 5))
   (segment (start 117.15 116.5) (end 120.07 116.5) (width 0.5) (layer F.Cu) (net 5))
@@
   (segment (start 130.834394 114.724394) (end 130.834394 111.796305) (width 0.5) (layer F.Cu) (net 5))
   (segment (start 133.49 117.38) (end 130.834394 114.724394) (width 0.5) (layer F.Cu) (net 5))
-  (segment (start 187.96 126.96) (end 188 127) (width 0.25) (layer F.Cu) (net 1))
-  (segment (start 193.04 121.92) (end 198 121.92) (width 0.5) (layer B.Cu) (net 1))
-  (segment (start 187.96 127) (end 193.04 121.92) (width 0.5) (layer B.Cu) (net 1))
-  (segment (start 184.570001 136.310001) (end 185.42 137.16) (width 0.25) (layer F.Cu) (net 3))
-  (segment (start 170.577994 121.724998) (end 182.372002 121.724998) (width 0.25) (layer F.Cu) (net 3))
-  (segment (start 183.194978 132.540852) (end 184.175013 133.520887) (width 0.25) (layer F.Cu) (net 3))
-  (segment (start 166.51 117.38) (end 167.309999 118.179999) (width 0.25) (layer F.Cu) (net 3))
-  (segment (start 184.175013 133.520887) (end 184.175013 135.915013) (width 0.25) (layer F.Cu) (net 3))
-  (segment (start 184.175013 135.915013) (end 184.570001 136.310001) (width 0.25) (layer F.Cu) (net 3))
-  (segment (start 182.372002 121.724998) (end 183.194978 122.547974) (width 0.25) (layer F.Cu) (net 3))
-  (segment (start 183.194978 122.547974) (end 183.194978 132.540852) (width 0.25) (layer F.Cu) (net 3))
-  (segment (start 167.309999 118.457003) (end 170.577994 121.724998) (width 0.25) (layer F.Cu) (net 3))
-  (segment (start 167.309999 118.179999) (end 167.309999 118.457003) (width 0.25) (layer F.Cu) (net 3))
   (segment (start 182.200001 134.100001) (end 182.6 134.5) (width 0.25) (layer F.Cu) (net 6))
   (segment (start 182.72 134.62) (end 182.6 134.5) (width 0.25) (layer B.Cu) (net 6))
@@
   (via (at 169 130.5) (size 0.8) (drill 0.4) (layers F.Cu B.Cu) (net 84))
   (segment (start 168.244999 131.255001) (end 169 130.5) (width 0.25) (layer B.Cu) (net 84))
-  (segment (start 138.65 130) (end 162.5 130) (width 0.25) (layer F.Cu) (net 85))
-  (segment (start 136.03 132.62) (end 138.65 130) (width 0.25) (layer F.Cu) (net 85))
-  (via (at 163 129.5) (size 0.8) (drill 0.4) (layers F.Cu B.Cu) (net 85))
-  (segment (start 162.5 130) (end 163 129.5) (width 0.25) (layer F.Cu) (net 85))
-  (via (at 169 129) (size 0.8) (drill 0.4) (layers F.Cu B.Cu) (net 85))
-  (segment (start 168.904999 128.904999) (end 169 129) (width 0.25) (layer B.Cu) (net 85))
-  (segment (start 163 129.5) (end 163.595001 128.904999) (width 0.25) (layer B.Cu) (net 85))
-  (segment (start 163.595001 128.904999) (end 168.904999 128.904999) (width 0.25) (layer B.Cu) (net 85))
   (segment (start 185 130) (end 185.46 129.54) (width 0.25) (layer B.Cu) (net 84))
   (segment (start 189.185001 127.649314) (end 188.519316 128.314999) (width 0.25) (layer F.Cu) (net 84))
@@
   (segment (start 185.42 129.54) (end 181.959953 129.54) (width 0.25) (layer B.Cu) (net 84))
   (segment (start 170 129.5) (end 181.354268 129.5) (width 0.25) (layer F.Cu) (net 84))
+  (segment (start 138.65 130) (end 162.5 130) (width 0.25) (layer F.Cu) (net 85))
+  (segment (start 136.03 132.62) (end 138.65 130) (width 0.25) (layer F.Cu) (net 85))
+  (via (at 163 129.5) (size 0.8) (drill 0.4) (layers F.Cu B.Cu) (net 85))
+  (segment (start 162.5 130) (end 163 129.5) (width 0.25) (layer F.Cu) (net 85))
+  (via (at 169 129) (size 0.8) (drill 0.4) (layers F.Cu B.Cu) (net 85))
+  (segment (start 168.904999 128.904999) (end 169 129) (width 0.25) (layer B.Cu) (net 85))
+  (segment (start 163 129.5) (end 163.595001 128.904999) (width 0.25) (layer B.Cu) (net 85))
+  (segment (start 163.595001 128.904999) (end 168.904999 128.904999) (width 0.25) (layer B.Cu) (net 85))
   (segment (start 189.685012 129.017069) (end 189.162081 129.54) (width 0.25) (layer F.Cu) (net 85))
   (segment (start 192.672996 119.38) (end 189.685012 122.367984) (width 0.25) (layer F.Cu) (net 85))
