File: CAD/mcu_controller/mcu_controller.sch (KiCad schematic (older format))
At the start: 75 parts

Commit message: finishes mcu controller schematic
Connections:
- net labels added: 3V3, MISO, MOSI, SCK
- wire segments 204 -> 258
- no-connect marks 4 -> 12

Commit message: progress on charge and output layout
Parts:
- removed J?: out2_fb, symbol Connector_Generic:Conn_01x05
- removed J?: out2_ch_en, symbol Connector_Generic:Conn_01x05
- removed R? (x4): 1K, symbol Device:R_Small
- removed R? (x4): 100, symbol Device:R_Small
- added D?: LED_Small, symbol Device:LED_Small
- added J?: Conn_02x05_Odd_Even, symbol Connector_Generic:Conn_02x05_Odd_Even
- added J?: out2_en, symbol Connector_Generic:Conn_01x02
- added R?: 1K, symbol Device:R_Small
- added R?: R_Small, symbol Device:R_Small
Connections:
- net labels removed: out2_ch1_en, out2_ch1_i, out2_ch2_en, out2_ch2_i, out2_ch3_en, out2_ch3_i, out2_ch4_en, out2_ch4_i
- wire segments 258 -> 253
- no-connect marks 12 -> 4

Commit message: finishes layout for mcu controller
Parts:
- removed C?: 0.1uF, symbol Device:C_Small
- removed D?: TL431DBV, Package_TO_SOT_SMD:SOT-23-5, symbol Reference_Voltage:TL431DBV
- removed J?: 3V3, symbol Connector_Generic:Conn_01x01
- removed J?: out2_en, symbol Connector_Generic:Conn_01x02
- removed JP?: UART_TX, symbol Device:Jumper_NO_Small
- removed JP?: UART_RX, symbol Device:Jumper_NO_Small
- removed R?: 1K, symbol Device:R_Small
- removed U?: ADuM1201AR, Package_SO:SOIC-8_3.9x4.9mm_P1.27mm, symbol Isolator:ADuM1201AR
- added D2: TL431DBZ, Package_TO_SOT_SMD:SOT-23, symbol Reference_Voltage:TL431DBZ
- added J10: out2_ch_en, Connector_PinSocket_2.54mm:PinSocket_1x05_P2.54mm_Vertical, symbol Connector_Generic:Conn_01x05
- added J7: out2_fb, Connector_PinSocket_2.54mm:PinSocket_1x05_P2.54mm_Vertical, symbol Connector_Generic:Conn_01x05
- added MK1, MK2, MK3, MK4: Mounting_Hole, MountingHole:MountingHole_4.3mm_M4, symbol Mechanical:Mounting_Hole
- added R15, R18, R7, R9: 100, Jumper:SolderJumper-2_P1.3mm_Open_RoundedPad1.0x1.5mm, symbol Device:R_Small
- added R24: R, Resistor_SMD:R_0603_1608Metric, symbol Device:R
- added R32, R33, R34, R35: 1K, Jumper:SolderJumper-2_P1.3mm_Open_RoundedPad1.0x1.5mm, symbol Device:R_Small
- added R45, R46, R47: 1K, Resistor_SMD:R_0603_1608Metric, symbol Device:R_Small
- C1, C3: renamed from C?; footprint (none) -> Capacitor_SMD:C_1206_3216Metric
- C2: renamed from C?; footprint (none) -> Capacitor_SMD:C_0603_1608Metric
- D1, D3: renamed from D?; footprint (none) -> LED_SMD:LED_0603_1608Metric
- J1, J2: renamed from J?; footprint (none) -> Connector_Phoenix_MC:PhoenixContact_MCV_1,5_2-G-5.08_1x02_P5.08mm_Vertical
- J11, J6, J9: renamed from J?; footprint (none) -> Connector_PinSocket_2.54mm:PinSocket_1x05_P2.54mm_Vertical
- J12, J13, J15, J19: renamed from J?; footprint (none) -> Connector_PinSocket_2.54mm:PinSocket_1x04_P2.54mm_Vertical
- J14: renamed from J?; value chrg3_ctrl -> chrg2_ctrl; footprint (none) -> Connector_PinSocket_2.54mm:PinSocket_1x04_P2.54mm_Vertical
- J16, J17: renamed from J?; footprint (none) -> Connector_PinSocket_2.54mm:PinSocket_1x02_P2.54mm_Vertical
- J20: renamed from J?; value Conn_02x05_Odd_Even -> UEXT; footprint (none) -> Connector_PinSocket_2.54mm:PinSocket_2x05_P2.54mm_Vertical
- J3, J4, J5: renamed from J?; footprint (none) -> Connector_PinSocket_2.54mm:PinSocket_1x03_P2.54mm_Vertical
- JP1, JP2: renamed from JP?; footprint (none) -> Jumper:SolderJumper-2_P1.3mm_Bridged_RoundedPad1.0x1.5mm
- R1, R10, R11, R12, R13, R14, R16, R17, R19, R2, R20, R21, R22, R23, R25, R26, R27, R3, R36, R37, R38, R39, R4, R40, R41, R42, R43, R44, R5, R6, R8: renamed from R?; footprint (none) -> Resistor_SMD:R_0603_1608Metric
- R28, R29, R30, R31: renamed from R?; footprint (none) -> Jumper:SolderJumper-2_P1.3mm_Open_RoundedPad1.0x1.5mm
- SW1: renamed from SW?; footprint (none) -> Connector_PinSocket_2.54mm:PinSocket_1x02_P2.54mm_Vertical
- U1: renamed from U?; footprint (none) -> Package_SO:SOIC-8_3.9x4.9mm_P1.27mm
- U2: renamed from U?; footprint (none) -> Package_TO_SOT_SMD:SOT-223-3_TabPin2
- U3: renamed from U?; footprint (none) -> teensy:Teensy30_31_32_LC
Connections:
- net labels added: A0, A1, A2, A3, A4, A5, A6, A7, A8, A9, BATT_IN, BATT_SW, RESET, RX, TX, out2_ch1_en, out2_ch1_i, out2_ch2_en, out2_ch2_i, out2_ch3_en, out2_ch3_i, out2_ch4_en, out2_ch4_i
- wire segments 253 -> 254
- no-connect marks 4 -> 9

Commit message: removes pin 17 connection to VIN on mcu controller
Connections:
- wire segments 254 -> 252
Changed lines of the file:
@@
 	8600 5850 9200 5850
-Wire Wire Line
-	8600 6350 8800 6350
-Wire Wire Line
-	8800 6350 8800 5350
 Wire Wire Line
 	6400 4150 6400 7250
 $Comp
-L power:+5V #PWR0129
-U 1 1 5B3D8697
-P 8800 5350
-F 0 "#PWR0129" H 8800 5200 50  0001 C CNN
-F 1 "+5V" H 8815 5523 50  0000 C CNN
-F 2 "" H 8800 5350 50  0001 C CNN
-F 3 "" H 8800 5350 50  0001 C CNN
-	1    8800 5350
-	1    0    0    -1
-$EndComp
-$Comp
 L power:GND #PWR0130
